File: arming_board.kicad_pcb (KiCad board)
At the start: 2 copper layers, 42 x 42 mm, 32 parts, among them IC1 CD4043BDR, J3 Conn_01x04, Q2 SQJ409EP

Commit message: fix mosfet
Parts:
- moved Q2 0.46 mm to (136.0, 120.8), turned to 0 degrees
Connections:
- Q2 pad 1: +BATT_ARM -> VCC
- Q2 pad 2: +BATT_ARM -> VCC
- Q2 pad 3: +BATT_ARM -> VCC
- Q2 pad 5: VCC -> +BATT_ARM
Routing:
- net Net-(Q2-G): track 13.3 -> 8.78 mm
- net +BATT_ARM: track 3.21 -> 4.68 mm
Other:
- board text added: "rev2"
- board text removed: "rev1"
